File: PICO-AT-softpower/PICO-AT.kicad_pcb (KiCad board)
At the start: 4 copper layers, 54.4 x 34.8 mm, 16 parts, among them IC1 MAX16054AZT+T, J1 09-48-1064, J2 09-48-1064, J3 87427-2402, U1 L7905

Commit message: Add files via upload
Connections:
- IC1 pad 6: /3.3V -> /5VSB
Routing:
- net /5VSB: track 0.00 -> 35.5 mm
- net /3.3V: track 7.95 -> 0.09 mm, vias 1 -> 0
