File: PICO-AT-softpower/PICO-AT.sch (KiCad schematic (older format))
At the start: 16 parts, among them IC1 MAX16054AZT+T, J1 09-48-1064, J2 09-48-1064, J3 87427-2402, J4 PWR_SW, U1 L7905

Commit message: Add files via upload
Connections:
- net 3.3V: no longer IC1.6 (VCC)
- net 5VSB: now also IC1.6 (VCC)
Changed lines of the file:
@@
 Connection ~ 5750 2150
 Text Label 7200 1950 0    50   ~ 0
-3.3V
+5VSB
 Wire Wire Line
 	7050 1950 7200 1950
